File: KiCad/Testbench/Shutdown_Circuit.kicad_sch (KiCad schematic)
At the start: 55 parts, among them J10 Conn_01x02_Pin, J11 Conn_01x02_Pin, J12 Conn_01x02_Pin, J13 Conn_01x02_Pin, J14 Conn_01x02_Pin, J15 Conn_01x02_Pin, J16 Conn_01x02_Pin, J17 Conn_01x02_Pin, J5 Conn_01x01_Pin, J6 Conn_02x05_Counter_Clockwise, J7 Conn_01x02_Pin, J8 Conn_01x02_Pin, J9 Conn_02x05_Counter_Clockwise

Commit message: PCB before first processing
Parts:
- removed D4, D5, D6: LED, LED_SMD:LED_0805_2012Metric_Pad1.15x1.40mm_HandSolder, symbol Device:LED
- removed R6, R7, R8: R1k1, Resistor_SMD:R_1206_3216Metric_Pad1.30x1.75mm_HandSolder, symbol Device:R
- added D11, D15, D16: LED, LED_SMD:LED_0805_2012Metric_Pad1.15x1.40mm_HandSolder, symbol Device:LED
- added R13, R17, R18: R1k1, Resistor_SMD:R_1206_3216Metric_Pad1.30x1.75mm_HandSolder, symbol Device:R
- renumbered D11 to D14, R13 to R16
Connections:
- net 1-A1: now also D10.2 (A)
- net 1-A3: now also D7.2 (A)
- net 1-B1: no longer D7.2 (A)
- net 1-B2: now also D11.2 (A)
- net 1-B3: no longer D8.2 (A)
- net 1-B4: now also D13.2 (A)
- net 1-C1: now also D8.2 (A)
- net 1-C2: no longer D12.2 (A)
- net 1-C3: now also D15.2 (A)
- net 1-C4: no longer D10.2 (A)
- net 1-D2: now also D9.2 (A)
- net 1-D4: now also D12.2 (A)
- net 1-E1: now also D16.2 (A)
- net 1-E2: no longer D14.2 (A)
- net 1-E3: now also D14.2 (A)
- net 1-E4: no longer D9.2 (A)
- net 1-F1: no longer D13.2 (A)
- net GND-LV_Unfiltered: now also R13.2, R17.2, R18.2
- new net: D15.1 (K), R17.1
- new net: D11.1 (K), R13.1
- new net: D16.1 (K), R18.1
Other:
- moved on the sheet: D14, R16
