File: KiCad/Testbench/Actuator.kicad_sch (KiCad schematic)
At the start: 7 parts, among them J1 Conn_02x03_Counter_Clockwise

Commit message: PCB before first processing
Parts:
- added D1, D3, D4: LED, LED_SMD:LED_0805_2012Metric_Pad1.15x1.40mm_HandSolder, symbol Device:LED
- added R1, R3, R4: R1k1, Resistor_SMD:R_1206_3216Metric_Pad1.30x1.75mm_HandSolder, symbol Device:R
- J1: footprint Connector_Molex:Molex_Mini-Fit_Jr_5566-06A_2x03_P4.20mm_Vertical -> Connector_Molex:Molex_Mini-Fit_Jr_5566-08A_2x04_P4.20mm_Vertical; symbol Connector_Generic:Conn_02x03_Counter_Clockwise -> Connector_Generic:Conn_02x04_Top_Bottom
- renumbered D1 to D2, D2 to D5, D3 to D6, R1 to R2, R2 to R5, R3 to R6
Connections:
- net 1-G3: now also J1.1 (Pin_1), R1.1; no longer J1.3 (Pin_3), J1.5 (Pin_5), J1.6 (Pin_6), R2.1
- net 2-B4: now also J1.6 (Pin_6); no longer J1.1 (Pin_1)
- net 2-E4: now also J1.5 (Pin_5); no longer J1.2 (Pin_2)
- net GND-LV_Unfiltered: now also J1.7 (Pin_7), D1.1 (K), D3.1 (K), D4.1 (K); no longer J1.4 (Pin_4)
- new net: D4.2 (A), R4.2
- new net: D3.2 (A), R3.2
- new net: D1.2 (A), R1.2
- new net 1-G4: J1.4 (Pin_4), R4.1
- new net 2-C4: J1.2 (Pin_2), R2.1
- new net 2-D4: J1.3 (Pin_3), R3.1
- no-connect marks 0 -> 1
Other:
- moved on the sheet: D2, R2

Commit message: After work 151024
Changed lines of the file:
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@@
 	(wire
 		(pts
-			(xy 140.97 137.16) (xy 140.97 146.05)
+			(xy 111.76 130.81) (xy 111.76 139.7)
 		)
 		(stroke
@@
 	)
 	(label "2-E3"
-		(at 140.97 137.16 0)
+		(at 111.76 130.81 0)
 		(fields_autoplaced yes)
 		(effects
@@
 	(symbol
 		(lib_id "power:GND")
-		(at 140.97 146.05 0)
+		(at 111.76 139.7 0)
 		(unit 1)
 		(exclude_from_sim no)
@@
 		(dnp no)
 		(property "Reference" "#PWR05"
-			(at 140.97 152.4 0)
+			(at 111.76 146.05 0)
 			(effects
 				(font
@@
 		)
 		(property "Value" "GND-LV_Unfiltered"
-			(at 132.08 150.114 0)
+			(at 102.87 143.764 0)
 			(effects
 				(font
@@
 		)
 		(property "Footprint" ""
-			(at 140.97 146.05 0)
+			(at 111.76 139.7 0)
 			(effects
 				(font
@@
 		)
 		(property "Datasheet" ""
-			(at 140.97 146.05 0)
+			(at 111.76 139.7 0)
 			(effects
 				(font
@@
 		)
 		(property "Description" "Power symbol creates a global label with name \"GND\" , ground"
-			(at 140.97 146.05 0)
-			(effects
-				(font
+			(at 111.76 139.7 0)
+			(effects
+				(font
