File: KiCad/Testbench/CAN.kicad_sch (KiCad schematic)
At the start: 10 parts, among them J2 Conn_02x02_Top_Bottom, J3 Conn_02x02_Top_Bottom, J4 Conn_02x02_Top_Bottom

Commit message: PCB before first processing
Parts:
- renumbered R4 to R7, R5 to R8
Changed lines of the file:
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@@
 		(on_board yes)
 		(dnp no)
-		(property "Reference" "R4"
+		(property "Reference" "R7"
 			(at 69.596 52.324 90)
 			(effects
@@
 			(project ""
 				(path "/7bff671f-2f7d-4dcb-82cb-7f168fb2ab46/91fc52e8-d123-4e03-9a67-b86afe193964"
-					(reference "R4")
+					(reference "R7")
 					(unit 1)
 				)
@@
 		(dnp no)
 		(fields_autoplaced yes)
-		(property "Reference" "#PWR05"
+		(property "Reference" "#PWR08"
 			(at 59.69 101.6 0)
 			(effects
@@
 			(project "Testbench"
 				(path "/7bff671f-2f7d-4dcb-82cb-7f168fb2ab46/91fc52e8-d123-4e03-9a67-b86afe193964"
-					(reference "#PWR05")
+					(reference "#PWR08")
 					(unit 1)
 				)
@@
 		(on_board yes)
 		(dnp no)
-		(property "Reference" "R5"
+		(property "Reference" "R8"
 			(at 208.28 50.8 90)
 			(effects
@@
 			(project ""
 				(path "/7bff671f-2f7d-4dcb-82cb-7f168fb2ab46/91fc52e8-d123-4e03-9a67-b86afe193964"
-					(reference "R5")
+					(reference "R8")
 					(unit 1)
 				)

Commit message: After work 151024
Other:
- note added: "Filtered GND for CAN"
Changed lines of the file:
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@@
+		)
+	)
+	(text "Filtered GND for CAN\n"
+		(exclude_from_sim no)
+		(at 68.072 71.882 0)
+		(effects
+			(font
+				(size 4 4)
+			)
 		)
 	)
